Commit message: Updated Dockerfile, added ros2_control test_hardware tag to URDF

File: myscarabot_ros/msb_description/xacro/scarabot.xacro (robot description, xacro)
@@ -114,8 +114,36 @@
     </visual>
   </link>
+  <!-- Add ros2_control tag -->
   <ros2_control name="myscarabot" type="system">
     <hardware>
-      <plugin>test_system</plugin>
+      <plugin>test_hardware_components/TestTwoJointSystem</plugin>
     </hardware>
+    <joint name="joint_1">
+      <command_interface name="position">
+        <param name="min">-2.356</param>
+        <param name="max">2.356</param>
+      </command_interface>
+      <state_interface name="position" />
+      <state_interface name="velocity" />
+      <state_interface name="effort"   />
+    </joint>
+    <joint name="joint_2">
+      <command_interface name="position">
+        <param name="min">-2.356</param>
+        <param name="max">2.356</param>
+      </command_interface>
+      <state_interface name="position" />
+      <state_interface name="velocity" />
+      <state_interface name="effort"   />
+    </joint>
+    <joint name="joint_3">
+      <command_interface name="position">
+        <param name="min">0.0</param>
+        <param name="max">0.4</param>
+      </command_interface>
+      <state_interface name="position" />
+      <state_interface name="velocity" />
+      <state_interface name="effort"   />
+    </joint>
   </ros2_control>
 </robot>

Commit message: Updated CMakeLists of msb_description to remove meshes folder

File: myscarabot_ros/msb_description/xacro/scarabot.xacro (robot description, xacro)
@@ -106,44 +106,27 @@
       <material name="black" />
     </visual>
+  </link>
+  <link name="link_4">
     <visual>
       <geometry>
         <cylinder radius="0.075" length="0.05" />
       </geometry>
-      <origin rpy="0 0 0" xyz="0 0 -0.175" />
+      <origin rpy="0 0 0" xyz="0 0 0" />
       <material name="black" />
     </visual>
+    <collision>
+      <geometry>
+        <cylinder radius="0.075" length="0.05" />
+      </geometry>
+      <origin rpy="0 0 0" xyz="0 0 0" />
+      <material name="black" />
+    </collision>
   </link>
-  <!-- Add ros2_control tag -->
-  <ros2_control name="myscarabot" type="system">
-    <hardware>
-      <plugin>test_hardware_components/TestTwoJointSystem</plugin>
-    </hardware>
-    <joint name="joint_1">
-      <command_interface name="position">
-        <param name="min">-2.356</param>
-        <param name="max">2.356</param>
-      </command_interface>
-      <state_interface name="position" />
-      <state_interface name="velocity" />
-      <state_interface name="effort"   />
-    </joint>
-    <joint name="joint_2">
-      <command_interface name="position">
-        <param name="min">-2.356</param>
-        <param name="max">2.356</param>
-      </command_interface>
-      <state_interface name="position" />
-      <state_interface name="velocity" />
-      <state_interface name="effort"   />
-    </joint>
-    <joint name="joint_3">
-      <command_interface name="position">
-        <param name="min">0.0</param>
-        <param name="max">0.4</param>
-      </command_interface>
-      <state_interface name="position" />
-      <state_interface name="velocity" />
-      <state_interface name="effort"   />
-    </joint>
-  </ros2_control>
+  <joint name="joint_4" type="revolute">
+    <parent link="link_3" />
+    <child link="link_4" />
+    <limit lower="-2.356" upper="2.356" effort="10.0" velocity="1.0"/>
+    <origin rpy="0 0 0" xyz="0 0 -0.175" />
+    <axis xyz="0 0 1" />
+  </joint>
 </robot>

Commit message: Reduced robot size, added collision geometry

File: myscarabot_ros/msb_description/xacro/scarabot.xacro (robot description, xacro)
@@ -1,22 +1,19 @@
 <robot name="scara_robot" xmlns:xacro="http://www.ros.org/wiki/xacro">
   <material name="black">
-    <color rgba="0 0 0 1.0" />
+    <color rgba="0.0 0.0 0.0 1.0" />
   </material>
   <material name="blue">
-    <color rgba="0 0 1 1.0" />
+    <color rgba="0.0 0.0 1.0 1.0" />
   </material>
   <material name="white">
-    <color rgba="1 1 1 1.0" />
+    <color rgba="1.0 1.0 1.0 1.0" />
   </material>
-  <link name="base_footprint"/>
-  <joint name="world" type="fixed">
-    <parent link="base_footprint"/>
-    <child link="base"/>
-    <origin rpy="0 0 0" xyz="0 0 0.1"/>
-  </joint>
+  <material name="red">
+    <color rgba="1.0 0.0 0.0 1.0" />
+  </material>
   <link name="base">
     <visual>
         <geometry>
-          <cylinder radius="0.2" length="0.2" />
+          <cylinder radius="0.1" length="0.05" />
         </geometry>
         <origin rpy="0 0 0" xyz="0 0 0" />
@@ -25,28 +22,27 @@
     <visual>
       <geometry>
-        <cylinder radius="0.1" length="0.4" />
+        <cylinder radius="0.05" length="0.3" />
       </geometry>
-      <origin rpy="0 0 0" xyz="0 0 0.2" />
+      <origin rpy="0 0 0" xyz="0 0 0.15" />
       <material name="blue" />
     </visual>
+    <collision>
+      <origin xyz="0.0 0.0 0.15" rpy="0.0 0.0 0.0" />
+      <geometry>
+        <cylinder radius="0.1" length="0.3" />
+      </geometry>
+    </collision>
   </link>
-  <joint name="joint_1" type="revolute">
-    <parent link="base" />
-    <child link="link_1" />
-    <limit lower="-2.356" upper="2.356" effort="10.0" velocity="1.0"/>
-    <origin rpy="0 0 0" xyz="0 0 0.3" />
-    <axis xyz="0 0 1" />
-  </joint>
   <link name="link_1">
     <visual>
       <geometry>
-        <box size="0.4 0.25 0.15" />
+        <box size="0.3 0.1 0.05" />
       </geometry>
-      <origin rpy="0 0 0" xyz="0.2 0 0" />
+      <origin rpy="0 0 0" xyz="0.15 0 0" />
       <material name="white"/>
     </visual>
     <visual>
       <geometry>
-        <cylinder radius="0.125" length="0.15" />
+        <cylinder radius="0.05" length="0.05" />
       </geometry>
       <origin rpy="0 0 0" xyz="0 0 0" />
@@ -55,28 +51,27 @@
     <visual>
       <geometry>
-        <cylinder radius="0.125" length="0.15" />
+        <cylinder radius="0.05" length="0.05" />
       </geometry>
-      <origin rpy="0 0 0" xyz="0.4 0 0" />
+      <origin rpy="0 0 0" xyz="0.3 0 0" />
       <material name="white"/>
     </visual>
+    <collision>
+      <origin xyz="0.15 0.0 0.0" rpy="0.0 0.0 0.0" />
+      <geometry>
+        <box size="0.4 0.1 0.05" />
+      </geometry>
+    </collision>
   </link>
-  <joint name="joint_2" type="revolute">
-    <parent link="link_1" />
-    <child link="link_2" />
-    <origin rpy="0 0 0" xyz="0.4 0 0.25" />
-    <limit lower="-2.356" upper="2.356" effort="10.0" velocity="1.0"/>
-    <axis xyz="0 0 1" />
-  </joint>
   <link name="link_2">
     <visual>
       <geometry>
-        <box size="0.4 0.25 0.35" />
+        <box size="0.3 0.1 0.15" />
       </geometry>
-      <origin rpy="0 0 0" xyz="0.2 0 0" />
+      <origin rpy="0 0 0" xyz="0.15 0 0" />
       <material name="white"/>
     </visual>
     <visual>
       <geometry>
-        <cylinder radius="0.125" length="0.35" />
+        <cylinder radius="0.05" length="0.15" />
       </geometry>
       <origin rpy="0 0 0" xyz="0 0 0" />
@@ -85,48 +80,75 @@
     <visual>
       <geometry>
-        <cylinder radius="0.125" length="0.35" />
+        <cylinder radius="0.05" length="0.15" />
       </geometry>
-      <origin rpy="0 0 0" xyz="0.4 0 0" />
+      <origin rpy="0 0 0" xyz="0.3 0 0" />
       <material name="white"/>
     </visual>
+    <collision>
+      <origin xyz="0.15 0.0 0.0" rpy="0.0 0.0 0.0" />
+      <geometry>
+        <box size="0.4 0.1 0.15" />
+      </geometry>
+    </collision>
   </link>
-  <joint name="joint_3" type="prismatic">
-    <parent link="link_2" />
-    <child link="link_3" />
-    <origin rpy="0 0 0" xyz="0.4 0 -0.05" />
-    <limit lower="0.0" upper="0.4" effort="10.0" velocity="1.0"/>
-    <axis xyz="0 0 -1" />
-  </joint>
   <link name="link_3">
     <visual>
       <geometry>
-        <cylinder radius="0.05" length="0.6" />
+        <cylinder radius="0.02" length="0.3" />
       </geometry>
       <origin rpy="0 0 0" xyz="0 0 0.1" />
       <material name="black" />
     </visual>
+    <collision>
+      <geometry>
+        <cylinder radius="0.02" length="0.3" />
+      </geometry>
+      <origin rpy="0 0 0" xyz="0 0 0.1" />
+      <material name="black" />
+    </collision>
   </link>
   <link name="link_4">
     <visual>
+      <origin xyz="0.0 0.0 0.0" rpy="0.0 0.0 0.0" />
       <geometry>
-        <cylinder radius="0.075" length="0.05" />
+        <cylinder radius="0.025" length="0.025"/>
       </geometry>
-      <origin rpy="0 0 0" xyz="0 0 0" />
       <material name="black" />
     </visual>
     <collision>
+      <origin xyz="0.0 0.0 0.0" rpy="0.0 0.0 0.0" />
       <geometry>
-        <cylinder radius="0.075" length="0.05" />
+        <cylinder radius="0.025" length="0.025"/>
       </geometry>
-      <origin rpy="0 0 0" xyz="0 0 0" />
-      <material name="black" />
+      <material name="red" />
     </collision>
   </link>
-  <joint name="joint_4" type="revolute">
+  <!-- JOINTS -->
+  <joint name="joint_1" type="revolute">
+    <parent link="base" />
+    <child link="link_1" />
+    <limit lower="-2.356" upper="2.356" effort="10.0" velocity="1.0"/>
+    <origin rpy="0 0 0" xyz="0 0 0.25" />
+    <axis xyz="0 0 1" />
+  </joint>
+  <joint name="joint_2" type="revolute">
+    <parent link="link_1" />
+    <child link="link_2" />
+    <origin rpy="0 0 0" xyz="0.3 0 0.05" />
+    <limit lower="-2.356" upper="2.356" effort="10.0" velocity="1.0"/>
+    <axis xyz="0 0 1" />
+  </joint>
+  <joint name="joint_3" type="prismatic">
+    <parent link="link_2" />
+    <child link="link_3" />
+    <origin rpy="0 0 0" xyz="0.3 0 -0.05" />
+    <limit lower="0.0" upper="0.2" effort="10.0" velocity="1.0"/>
+    <axis xyz="0 0 -1" />
+  </joint>
+  <joint name="joint_4" type="continuous">
     <parent link="link_3" />
     <child link="link_4" />
-    <limit lower="-2.356" upper="2.356" effort="10.0" velocity="1.0"/>
-    <origin rpy="0 0 0" xyz="0 0 -0.175" />
-    <axis xyz="0 0 1" />
+    <origin rpy="0.0 0.0 0.0" xyz="0.0 0.0 -0.05" />
+    <axis xyz="0.0 0.0 1.0"/>
   </joint>
 </robot>

Commit message: Added gazebo integration

File: myscarabot_ros/msb_description/xacro/scarabot.xacro (robot description, xacro)
@@ -1,15 +1,6 @@
 <robot name="scara_robot" xmlns:xacro="http://www.ros.org/wiki/xacro">
-  <material name="black">
-    <color rgba="0.0 0.0 0.0 1.0" />
-  </material>
-  <material name="blue">
-    <color rgba="0.0 0.0 1.0 1.0" />
-  </material>
-  <material name="white">
-    <color rgba="1.0 1.0 1.0 1.0" />
-  </material>
-  <material name="red">
-    <color rgba="1.0 0.0 0.0 1.0" />
-  </material>
+  <xacro:include filename="gazebo_references.xacro" />
+  <!-- LINKS -->
+  <link name="base_footprint" />
   <link name="base">
     <visual>
@@ -33,4 +24,9 @@
       </geometry>
     </collision>
+    <inertial>
+      <origin xyz="0.0 0.0 0.0" rpy="0.0 0.0 0.0" />
+      <mass value="10.0"/>
+      <inertia ixx="0.0228" ixy="0.0" ixz="0.0" iyy="0.0228" iyz="0.0" izz="0.0006" />
+    </inertial>
   </link>
   <link name="link_1">
@@ -62,4 +58,9 @@
       </geometry>
     </collision>
+    <inertial>
+      <origin xyz="0.0 0.0 0.0" rpy="0.0 0.0 0.0" />
+      <mass value="5.0" />
+      <inertia ixx="0.005208" ixy="0.0" ixz="0.0" iyy="0.03854" iyz="0.0" izz="0.041667" />
+    </inertial>
   </link>
   <link name="link_2">
@@ -90,5 +91,11 @@
         <box size="0.4 0.1 0.15" />
       </geometry>
+      <material name="red" />
     </collision>
+    <inertial>
+      <origin xyz="0.0 0.0 0.0" rpy="0.0 0.0 0.0" />
+      <mass value="3.5"/>
+      <inertia ixx="0.02708" ixy="0.0" ixz="0.0" iyy="0.09375" iyz="0.0" izz="0.08333" />
+    </inertial>
   </link>
   <link name="link_3">
@@ -105,6 +112,11 @@
       </geometry>
       <origin rpy="0 0 0" xyz="0 0 0.1" />
-      <material name="black" />
+      <material name="red" />
     </collision>
+    <inertial>
+      <origin xyz="0.0 0.0 0.0" rpy="0.0 0.0 0.0" />
+      <mass value="0.5"/>
+      <inertia ixx="0.0228" ixy="0.0" ixz="0.0" iyy="0.0228" iyz="0.0" izz="0.0006" />
+    </inertial>
   </link>
   <link name="link_4">
@@ -123,6 +135,16 @@
       <material name="red" />
     </collision>
+    <inertial>
+      <origin xyz="0.0 0.0 0.0" rpy="0.0 0.0 0.0" />
+      <mass value="0.5"/>
+      <inertia ixx="0.000625" ixy="0.0" ixz="0.0" iyy="0.000625" iyz="0.0" izz="0.0009375" />
+    </inertial>
   </link>
   <!-- JOINTS -->
+  <joint name="footprint" type="fixed">
+    <parent link="base_footprint" />
+    <child link="base"/>
+    <origin xyz="0.0 0.0 0.025" rpy="0.0 0.0 0.0" />
+  </joint>
   <joint name="joint_1" type="revolute">
     <parent link="base" />
